File: robot.kicad_pcb (KiCad board)
At the start: 2 copper layers, 56.3 x 118.2 mm, 87 parts, among them J1 PCA9865 2, J10 Servo pwr, J11 Vin, J12 I2C, J13 VCC, J14 +5V, J2 I2S, J3 Programming, J4 IMU, J5 Switches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

Commit message: Finished routing board revision 3: ready for first PCB run.
Parts:
- added J15: USB_B_Micro, Connector_USB:USB_Micro-B_Amphenol_10104110_Horizontal, F.Cu at (100.5, 127.0)
- added TP5: SCL_1, TestPoint:TestPoint_Pad_D2.0mm, F.Cu at (142.7, 145.8)
- added TP6: SDA_1, TestPoint:TestPoint_Pad_D2.0mm, F.Cu at (135.1, 145.8)
- J6: footprint Connector_PinSocket_2.54mm:PinSocket_1x09_P2.54mm_Vertical -> Connector_PinSocket_2.54mm:PinSocket_2x04_P2.54mm_Vertical
- TP2, TP3, TP4: moved to B.Cu
- moved TP4 40.9 mm to (130.8, 159.5), turned to 180 degrees
- moved TP3 39.4 mm to (130.8, 165.6), turned to 180 degrees
- moved TP2 39.4 mm to (130.8, 162.6), turned to 180 degrees
- moved D2 39.4 mm to (103.9, 134.1), turned to 180 degrees
- moved R8 38.6 mm to (103.9, 137.7)
- moved D3 38.3 mm to (137.7, 113.8), turned to 0 degrees
- moved SW6 34.8 mm to (114.8, 128.0), turned to -90 degrees
- moved SW4 34.4 mm to (135.1, 128.0), turned to -90 degrees
- moved R28 32.9 mm to (139.2, 119.4), turned to 90 degrees
- moved R5 17.2 mm to (115.3, 97.5), turned to 0 degrees
- moved R11 16.9 mm to (103.9, 106.3)
- moved SW2 16.8 mm to (126.0, 128.0)
- moved R27 12.3 mm to (125.5, 121.5), turned to 0 degrees
- moved J6 11.4 mm to (99.0, 118.1)
- moved C2 9.41 mm to (119.9, 127.0), turned to 180 degrees
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Connections:
- J2 pad 4: Net-(J2-Pin_4) -> /Ports/AUDIO GAIN
- J6 pad 1: IO_0 -> /Ports/AUDIO GAIN
- J6 pad 2: IO_11 -> IO_16
- J6 pad 3: IO_16 -> IO_40
- J6 pad 4: IO_40 -> IO_42
- J6 pad 5: IO_42 -> IO_45
- J6 pad 6: IO_45 -> IO_46
- J6 pad 7: IO_46 -> GND
- J6 pad 8: GND -> VCC
- JP5 pad 2: Net-(J2-Pin_4) -> /Ports/AUDIO GAIN
- R11 pad 2: Net-(J2-Pin_4) -> /Ports/AUDIO GAIN
Routing:
- net GND: track 376.5 -> 876.2 mm, vias 8 -> 21
- net VCC: track 158.3 -> 310.0 mm, vias 5 -> 6
- net WIRE_1_SCL: track 25.7 -> 126.6 mm, vias 0 -> 4
- net WIRE_0_SDA: track 0.00 -> 68.5 mm, vias 0 -> 2
- net /SWITCH_6: track 0.00 -> 56.2 mm, vias 0 -> 1
- net WIRE_0_SCL: track 12.4 -> 64.9 mm, vias 0 -> 3
- net +BATT: track 35.3 -> 86.3 mm
- net IO_45: track 0.00 -> 50.8 mm, vias 0 -> 1
- net ONEWIRE_BUS: track 38.5 -> 88.0 mm, vias 2 -> 3
- net /SWITCH_3: track 0.00 -> 48.1 mm
- net IO_40: track 0.00 -> 44.2 mm, vias 0 -> 3
- net IO_46: track 0.00 -> 42.5 mm, vias 0 -> 1
- net /SWITCH_7: track 0.00 -> 41.4 mm, vias 0 -> 1
- net IO_42: track 0.00 -> 38.9 mm, vias 0 -> 1
- net /SWITCH_2: track 0.00 -> 37.6 mm, vias 0 -> 1
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- added copper zone on B.Cu, net GND
- added copper zone on F.Cu, net GND
Other:
- board text added: "Combine +5V"
